File: keypad-pcb.kicad_pcb (KiCad board)
At the start: 2 copper layers, 24 parts, among them SW1 SW_Push, U1 ATmega32U4-A, Y1 16MHz

Commit message: More Wiring
Parts:
- moved C2 31.3 mm to (90.5, 40.5), turned to 0 degrees
- moved Y1 28.0 mm to (90.5, 36.5), turned to 90 degrees
- moved C3 25.8 mm to (90.5, 32.5), turned to 180 degrees
- moved C7 23.8 mm to (97.6, 47.6)
- moved C4 23.0 mm to (100.8, 45.2)
- moved C1 20.1 mm to (106.4, 49.2)
- moved SW1 19.2 mm to (98.4, 21.4), turned to 90 degrees
- moved C5 19.2 mm to (101.6, 48.4)
- moved R3 18.6 mm to (99.2, 30.2), turned to 90 degrees
- moved C6 12.9 mm to (104.8, 23.0)
- moved USB1 4.51 mm to (108.0, 14.6)
- moved R2 3.33 mm to (107.2, 22.8)
- moved R1 3.03 mm to (109.5, 22.8)
- moved F1 2.93 mm to (111.9, 23.6)
- moved U1 1.21 mm to (108.0, 33.3), turned to -90 degrees
Routing:
- net GND: track 0.55 -> 19.4 mm
- net Net-(R3-Pad2): track 0.00 -> 9.21 mm
- net +5V: track 0.00 -> 6.10 mm
- net Net-(C6-Pad1): track 0.00 -> 5.21 mm
- net Net-(R2-Pad2): track 0.00 -> 4.95 mm
- net Net-(R1-Pad2): track 0.00 -> 4.29 mm
- net Net-(C2-Pad2): track 0.00 -> 2.96 mm
- net Net-(C3-Pad2): track 0.00 -> 2.91 mm
- net D+: track 5.38 -> 3.14 mm
- net D-: track 5.07 -> 4.47 mm
